File: Hardware/SparkFun_LilyPad-Switched-Battery.brd (EAGLE design)
At the start: 29.4 x 29.2 mm, 11 parts

Commit message: updated board and sch files
Parts:
- removed U$8: CREATIVE_COMMONS, SparkFun-Aesthetics:CREATIVE_COMMONS
- added FRAME1: FRAME-LETTER, SparkFun-Aesthetics:CREATIVE_COMMONS
- added LOGO1: SFE_LOGO_FLAME.1_INCH, SparkFun-Aesthetics:SFE_LOGO_FLAME_.1
- BAT1: value (none) -> 20mm coincell
- JP1, JP2: device SparkFun:MICRO-FIDUCIAL -> SparkFun-Aesthetics:MICRO-FIDUCIAL
- S1: value (none) -> Switch
- moved JP1 9.67 mm to (-14.0, -8.89)
- moved U$7 3.44 mm to (-13.1, 0.32)
- moved JP2 1.27 mm to (3.81, 13.0)
- renumbered U$1 to ST1, U$2 to ST3, U$3 to ST2, U$4 to ST4
Connections:
- net N$2: now also BAT1.NEGATIVE; no longer BAT1.2
- net N$3: now also BAT1.POSITIVE@1, BAT1.POSITIVE@2, BAT1.POSITIVE@3, BAT1.POSITIVE@4; no longer BAT1.1, BAT1.3, BAT1.P$1, BAT1.P$2
Other:
- board text added: "Coin Cell Battery Holder"

Commit message: Updated Board and Schematic files
Parts:
- added U$1: REVISION, SparkFun-Aesthetics:REVISION
- moved FRAME1 92.0 mm to (-21.8, -10.2)
- moved U$7 42.3 mm to (20.6, 25.8), turned to 0 degrees
- moved JP1 39.9 mm to (6.35, 25.4), turned to 270 degrees
- moved S1 39.2 mm to (15.2, 25.8), turned to 180 degrees
- moved ST4 38.7 mm to (25.3, 22.7), turned to 137 degrees
- moved ST3 36.4 mm to (4.57, 22.7), turned to 223 degrees
- moved LOGO1 34.9 mm to (11.4, 24.2), turned to 0 degrees
- moved JP2 25.0 mm to (28.2, 7.62), turned to 270 degrees
- moved U$5 24.4 mm to (15.2, 15.2), turned to 0 degrees
- moved BAT1 19.1 mm to (15.2, 11.4), turned to 0 degrees
- moved ST2 16.4 mm to (24.0, 2.67), turned to 43 degrees
- moved ST1 11.7 mm to (6.48, 2.67), turned to 317 degrees
Routing:
- net N$1: track 22.9 -> 24.8 mm
- net N$2: track 26.1 -> 24.9 mm
Other:
- board size 29.4 x 29.2 mm -> 29.8 x 29.7 mm
- board text added: "Jim Lindblom"
- board text added: "Mary West"
