File: Hardware/SparkFun_LilyPad-Switched-Battery.sch (EAGLE design)
At the start: 11 parts

Commit message: updated board and sch files
Parts:
- removed U$8: CREATIVE_COMMONS, SparkFun-Aesthetics:CREATIVE_COMMONS
- added FRAME1: FRAME-LETTER, SparkFun-Aesthetics:FRAME-LETTER
- added LOGO1: SFE_LOGO_FLAME.1_INCH, SparkFun-Aesthetics:SFE_LOGO_FLAME.1_INCH
- BAT1: value (none) -> 20mm coincell
- JP1, JP2: device SparkFun:FIDUCIALUFIDUCIAL -> SparkFun-Aesthetics:FIDUCIALUFIDUCIAL
- S1: value (none) -> Switch
- renumbered U$1 to ST1, U$2 to ST3, U$3 to ST2, U$4 to ST4
Other:
- note added: "v14"
- note removed: "LilyPad - LED"
- note removed: "v12"
Changed lines of the file:
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@@
 <?xml version="1.0" encoding="utf-8"?>
 <!DOCTYPE eagle SYSTEM "eagle.dtd">
-<eagle version="7.2.0">
+<eagle version="7.5.0">
 <drawing>
 <settings>
@@
 <layer number="54" name="bGND_GNDA" color="1" fill="9" visible="no" active="no"/>
 <layer number="56" name="wert" color="7" fill="1" visible="no" active="no"/>
+<layer number="57" name="tCAD" color="7" fill="1" visible="no" active="no"/>
+<layer number="59" name="tCarbon" color="7" fill="1" visible="no" active="no"/>
+<layer number="60" name="bCarbon" color="7" fill="1" visible="no" active="no"/>
+<layer number="90" name="Modules" color="5" fill="1" visible="yes" active="yes"/>
 <layer number="91" name="Nets" color="2" fill="1" visible="yes" active="yes"/>
 <layer number="92" name="Busses" color="1" fill="1" visible="yes" active="yes"/>
@@
 <layer number="97" name="Info" color="7" fill="1" visible="yes" active="yes"/>
 <layer number="98" name="Guide" color="6" fill="1" visible="yes" active="yes"/>
+<layer number="99" name="SpiceOrder" color="7" fill="1" visible="no" active="no"/>
 <layer number="100" name="Muster" color="7" fill="1" visible="no" active="no"/>
 <layer number="101" name="Patch_Top" color="12" fill="4" visible="yes" active="yes"/>
@@
 <layer number="106" name="bPlate" color="7" fill="1" visible="yes" active="yes"/>
 <layer number="107" name="Crop" color="7" fill="1" visible="yes" active="yes"/>
+<layer number="108" name="tplace-old" color="10" fill="1" visible="yes" active="yes"/>
+<layer number="109" name="ref-old" color="11" fill="1" visible="yes" active="yes"/>
+<layer number="110" name="fp0" color="7" fill="1" visible="yes" active="yes"/>
+<layer number="111" name="LPC17xx" color="7" fill="1" visible="yes" active="yes"/>
+<layer number="112" name="tSilk" color="7" fill="1" visible="yes" active="yes"/>
+<layer number="113" name="IDFDebug" color="4" fill="1" visible="yes" active="yes"/>
 <layer number="116" name="Patch_BOT" color="9" fill="4" visible="yes" active="yes"/>
 <layer number="121" name="_tsilk" color="7" fill="1" visible="yes" active="yes"/>
 <layer number="122" name="_bsilk" color="7" fill="1" visible="yes" active="yes"/>
+<layer number="123" name="tTestmark" color="7" fill="1" visible="yes" active="yes"/>
+<layer number="124" name="bTestmark" color="7" fill="1" visible="yes" active="yes"/>
 <layer number="125" name="_tNames" color="7" fill="1" visible="no" active="yes"/>
+<layer number="126" name="_bNames" color="7" fill="1" visible="yes" active="yes"/>
+<layer number="127" name="_tValues" color="7" fill="1" visible="yes" active="yes"/>
+<layer number="128" name="_bValues" color="7" fill="1" visible="yes" active="yes"/>
+<layer number="129" name="Mask" color="7" fill="1" visible="yes" active="yes"/>
+<layer number="131" name="tAdjust" color="7" fill="1" visible="yes" active="yes"/>
+<layer number="132" name="bAdjust" color="7" fill="1" visible="yes" active="yes"/>
 <layer number="144" name="Drill_legend" color="7" fill="1" visible="yes" active="yes"/>
+<layer number="150" name="Notes" color="7" fill="1" visible="yes" active="yes"/>
 <layer number="151" name="HeatSink" color="7" fill="1" visible="yes" active="yes"/>
+<layer number="152" name="_bDocu" color="7" fill="1" visible="yes" active="yes"/>
+<layer number="153" name="FabDoc1" color="7" fill="1" visible="yes" active="yes"/>
+<layer number="154" name="FabDoc2" color="7" fill="1" visible="yes" active="yes"/>
+<layer number="155" name="FabDoc3" color="7" fill="1" visible="yes" active="yes"/>
+<layer number="199" name="Contour" color="7" fill="1" visible="yes" active="yes"/>
 <layer number="200" name="200bmp" color="1" fill="10" visible="no" active="no"/>
 <layer number="201" name="201bmp" color="2" fill="1" visible="no" active="no"/>
@@
 <layer number="223" name="223bmp" color="24" fill="1" visible="no" active="no"/>
 <layer number="224" name="224bmp" color="25" fill="1" visible="no" active="no"/>
+<layer number="225" name="225bmp" color="7" fill="1" visible="yes" active="yes"/>
+<layer number="226" name="226bmp" color="7" fill="1" visible="yes" active="yes"/>
+<layer number="227" name="227bmp" color="7" fill="1" visible="yes" active="yes"/>
+<layer number="228" name="228bmp" color="7" fill="1" visible="yes" active="yes"/>
+<layer number="229" name="229bmp" color="7" fill="1" visible="yes" active="yes"/>
+<layer number="230" name="230bmp" color="7" fill="1" visible="yes" active="yes"/>
+<layer number="231" name="231bmp" color="7" fill="1" visible="yes" active="yes"/>
+<layer number="248" name="Housing" color="7" fill="1" visible="yes" active="yes"/>
+<layer number="249" name="Edge" color="7" fill="1" visible="yes" active="yes"/>
 <layer number="250" name="Descript" color="3" fill="1" visible="no" active="no"/>
 <layer number="251" name="SMDround" color="12" fill="11" visible="no" active="no"/>
 <layer number="254" name="cooling" color="7" fill="1" visible="yes" active="yes"/>
+<layer number="255" name="routoute" color="7" fill="1" visible="yes" active="yes"/>
 </layers>
-<schematic xreflabel="%F%N/%S" xrefpart="/%S">
+<schematic xreflabel="%F%N/%S" xrefpart="/%S.%C%R">
 <attributes>
 </attributes>
@@
 </classes>
 <parts>
-<part name="FRAME1" library="SparkFun" deviceset="FRAME-LETTER" device=""/>
-<part name="U$1" library="LilyPad-Wearables" deviceset="SEWTAP" device="6"/>
-<part name="U$2" library="LilyPad-Wearables" deviceset="SEWTAP" device="6"/>
-<part name="U$3" library="LilyPad-Wearables" deviceset="SEWTAP" device="6"/>
-<part name="U$4" library="LilyPad-Wearables" deviceset="SEWTAP" device="6"/>
+<part name="FRAME1" library="SparkFun-Aesthetics" deviceset="FRAME-LETTER" device=""/>
+<part name="ST1" library="LilyPad-Wearables" deviceset="SEWTAP" device="6"/>
+<part name="ST3" library="LilyPad-Wearables" deviceset="SEWTAP" device="6"/>
+<part name="ST2" library="LilyPad-Wearables" deviceset="SEWTAP" device="6"/>
+<part name="ST4" library="LilyPad-Wearables" deviceset="SEWTAP" device="6"/>
 <part name="U$5" library="LilyPad-Wearables" deviceset="LOGO-LP" device="LP"/>
-<part name="S1" library="SparkFun" deviceset="SWITCH-SPST" device="SMD"/>
-<part name="BAT1" library="SparkFun-Electromechanical" deviceset="BATTERY" device="20MM_4LEGS"/>
+<part name="S1" library="SparkFun" deviceset="SWITCH-SPST" device="SMD" value="Switch"/>
+<part name="BAT1" library="SparkFun-Electromechanical" deviceset="BATTERY" device="20MM_4LEGS" value="20mm coincell"/>
 <part name="U$7" library="SparkFun-Aesthetics" deviceset="OSHW-LOGO" device="S"/>
-<part name="U$8" library="SparkFun-Aesthetics" deviceset="CREATIVE_COMMONS" device=""/>
-<part name="JP1" library="SparkFun" deviceset="FIDUCIAL" device="UFIDUCIAL"/>
-<part name="JP2" library="SparkFun" deviceset="FIDUCIAL" device="UFIDUCIAL"/>
+<part name="JP1" library="SparkFun-Aesthetics" deviceset="FIDUCIAL" device="UFIDUCIAL"/>
+<part name="JP2" library="SparkFun-Aesthetics" deviceset="FIDUCIAL" device="UFIDUCIAL"/>
+<part name="LOGO1" library="SparkFun-Aesthetics" deviceset="SFE_LOGO_FLAME" device=".1_INCH"/>
 </parts>
 <sheets>
 <sheet>
 <plain>
-<text x="154.94" y="27.94" size="3.175" layer="94">LilyPad - LED</text>
-<text x="43.18" y="10.16" size="1.778" layer="97">Jim Lindblom</text>
-<text x="238.76" y="7.62" size="1.778" layer="94">v12</text>
+<text x="170.942" y="11.684" size="1.778" layer="94">Jim Lindblom</text>
+<text x="238.76" y="7.62" size="1.778" layer="94">v14</text>
 </plain>
 <instances>
 <instance part="FRAME1" gate="G$1" x="0" y="0"/>
-<instance part="FRAME1" gate="G$2" x="147.32" y="0"/>
-<instance part="U$1" gate="G$1" x="127" y="99.06"/>
-<instance part="U$2" gate="G$1" x="88.9" y="96.52" rot="R180"/>
-<instance part="U$3" gate="G$1" x="127" y="93.98"/>
-<instance part="U$4" gate="G$1" x="88.9" y="91.44" rot="R180"/>
+<instance part="FRAME1" gate="V" x="147.32" y="0"/>
+<instance part="ST1" gate="G$1" x="127" y="99.06" smashed="yes">
+<attribute name="NAME" x="129.54" y="99.06" size="1.778" layer="95"/>
+</instance>
+<instance part="ST3" gate="G$1" x="88.9" y="96.52" smashed="yes" rot="R180">
+<attribute name="NAME" x="86.36" y="96.52" size="1.778" layer="95" rot="R180"/>
+</instance>
+<instance part="ST2" gate="G$1" x="127" y="93.98" smashed="yes">
+<attribute name="NAME" x="129.54" y="93.98" size="1.778" layer="95"/>
+</instance>
+<instance part="ST4" gate="G$1" x="88.9" y="91.44" smashed="yes" rot="R180">
+<attribute name="NAME" x="86.36" y="91.44" size="1.778" layer="95" rot="R180"/>
+</instance>
 <instance part="U$5" gate="G$1" x="236.22" y="17.78"/>
 <instance part="S1" gate="1" x="104.14" y="96.52" rot="R180"/>
 <instance part="BAT1" gate="G$1" x="114.3" y="96.52"/>
-<instance part="U$7" gate="G$1" x="12.7" y="12.7"/>
-<instance part="U$8" gate="G$1" x="25.4" y="10.16"/>
+<instance part="U$7" gate="G$1" x="233.68" y="48.26"/>
 <instance part="JP1" gate="G$1" x="236.22" y="30.48"/>
 <instance part="JP2" gate="G$1" x="243.84" y="30.48"/>
+<instance part="LOGO1" gate="G$1" x="215.9" y="40.64"/>
 </instances>
 <busses>
@@
 <wire x1="121.92" y1="93.98" x2="121.92" y2="96.52" width="0.1524" layer="91"/>
 <junction x="121.92" y="96.52"/>
-<pinref part="U$1" gate="G$1" pin="1"/>
-<pinref part="U$3" gate="G$1" pin="1"/>
+<pinref part="ST1" gate="G$1" pin="1"/>
+<pinref part="ST2" gate="G$1" pin="1"/>
 <pinref part="BAT1" gate="G$1" pin="-"/>
 </segment>
@@
 <wire x1="99.06" y1="93.98" x2="93.98" y2="93.98" width="0.1524" layer="91"/>
 <junction x="93.98" y="93.98"/>
-<pinref part="U$2" gate="G$1" pin="1"/>
-<pinref part="U$4" gate="G$1" pin="1"/>
+<pinref part="ST3" gate="G$1" pin="1"/>
+<pinref part="ST4" gate="G$1" pin="1"/>
 <pinref part="S1" gate="1" pin="O"/>
 </segment>

Commit message: Updated Board and Schematic files
Parts:
- added U$1: REVISION, SparkFun-Aesthetics:REVISION
Other:
- note added: "Mary West"
- note added: "v15"
- note removed: "v14"
Changed lines of the file:
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@@
 <part name="JP2" library="SparkFun-Aesthetics" deviceset="FIDUCIAL" device="UFIDUCIAL"/>
 <part name="LOGO1" library="SparkFun-Aesthetics" deviceset="SFE_LOGO_FLAME" device=".1_INCH"/>
+<part name="U$1" library="SparkFun-Aesthetics" deviceset="REVISION" device=""/>
 </parts>
 <sheets>
 <sheet>
 <plain>
-<text x="170.942" y="11.684" size="1.778" layer="94">Jim Lindblom</text>
-<text x="238.76" y="7.62" size="1.778" layer="94">v14</text>
+<text x="170.942" y="11.684" size="2.54" layer="94" font="vector">Jim Lindblom</text>
+<text x="238.76" y="7.62" size="1.778" layer="94">v15</text>
+<text x="177.8" y="7.62" size="2.54" layer="94" font="vector">Mary West </text>
 </plain>
 <instances>
@@
 <instance part="JP2" gate="G$1" x="243.84" y="30.48"/>
 <instance part="LOGO1" gate="G$1" x="215.9" y="40.64"/>
+<instance part="U$1" gate="G$1" x="149.86" y="7.62"/>
 </instances>
 <busses>

Commit message: updated board and schematic files
Parts:
- removed S1: Switch, SparkFun:SWITCH-SPSTSMD
- added S2: (no value), SparkFun-Electromechanical:SWITCH-SPDTSMD
Connections:
- net N$1: now also S2.O; no longer S1.O
- net N$3: now also S2.P; no longer S1.P
Changed lines of the file:
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@@
 <part name="ST4" library="LilyPad-Wearables" deviceset="SEWTAP" device="6"/>
 <part name="U$5" library="LilyPad-Wearables" deviceset="LOGO-LP" device="LP"/>
-<part name="S1" library="SparkFun" deviceset="SWITCH-SPST" device="SMD" value="Switch"/>
 <part name="BAT1" library="SparkFun-Electromechanical" deviceset="BATTERY" device="20MM_4LEGS" value="20mm coincell"/>
 <part name="U$7" library="SparkFun-Aesthetics" deviceset="OSHW-LOGO" device="S"/>
@@
 <part name="LOGO1" library="SparkFun-Aesthetics" deviceset="SFE_LOGO_FLAME" device=".1_INCH"/>
 <part name="U$1" library="SparkFun-Aesthetics" deviceset="REVISION" device=""/>
+<part name="S2" library="SparkFun-Electromechanical" deviceset="SWITCH-SPDT" device="SMD"/>
 </parts>
 <sheets>
@@
 </instance>
 <instance part="U$5" gate="G$1" x="236.22" y="17.78"/>
-<instance part="S1" gate="1" x="104.14" y="96.52" rot="R180"/>
 <instance part="BAT1" gate="G$1" x="114.3" y="96.52"/>
 <instance part="U$7" gate="G$1" x="233.68" y="48.26"/>
@@
 <instance part="LOGO1" gate="G$1" x="215.9" y="40.64"/>
 <instance part="U$1" gate="G$1" x="149.86" y="7.62"/>
+<instance part="S2" gate="1" x="104.14" y="96.52" rot="R180"/>
 </instances>
 <busses>
@@
 <pinref part="ST3" gate="G$1" pin="1"/>
 <pinref part="ST4" gate="G$1" pin="1"/>
-<pinref part="S1" gate="1" pin="O"/>
+<pinref part="S2" gate="1" pin="O"/>
 </segment>
 </net>
@@
 <segment>
 <wire x1="106.68" y1="96.52" x2="109.22" y2="96.52" width="0.1524" layer="91"/>
-<pinref part="S1" gate="1" pin="P"/>
 <pinref part="BAT1" gate="G$1" pin="+"/>
+<pinref part="S2" gate="1" pin="P"/>
 </segment>
 </net>

Commit message: Updated Board and Schematic files per QC
Parts:
- renumbered S2 to S1
Changed lines of the file:
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@@
 <part name="LOGO1" library="SparkFun-Aesthetics" deviceset="SFE_LOGO_FLAME" device=".1_INCH"/>
 <part name="U$1" library="SparkFun-Aesthetics" deviceset="REVISION" device=""/>
-<part name="S2" library="SparkFun-Electromechanical" deviceset="SWITCH-SPDT" device="SMD"/>
+<part name="S1" library="SparkFun-Electromechanical" deviceset="SWITCH-SPDT" device="SMD"/>
 </parts>
 <sheets>
@@
 <instance part="LOGO1" gate="G$1" x="215.9" y="40.64"/>
 <instance part="U$1" gate="G$1" x="149.86" y="7.62"/>
-<instance part="S2" gate="1" x="104.14" y="96.52" rot="R180"/>
+<instance part="S1" gate="1" x="104.14" y="96.52" rot="R180"/>
 </instances>
 <busses>
@@
 <pinref part="ST3" gate="G$1" pin="1"/>
 <pinref part="ST4" gate="G$1" pin="1"/>
-<pinref part="S2" gate="1" pin="O"/>
+<pinref part="S1" gate="1" pin="O"/>
 </segment>
 </net>
@@
 <wire x1="106.68" y1="96.52" x2="109.22" y2="96.52" width="0.1524" layer="91"/>
 <pinref part="BAT1" gate="G$1" pin="+"/>
-<pinref part="S2" gate="1" pin="P"/>
+<pinref part="S1" gate="1" pin="P"/>
 </segment>
 </net>
