File: Hardware/SparkFun_LilyPad-Switched-Battery_StakingVias_LargePads.brd (EAGLE design)
At the start: 30.2 x 30 mm, 13 parts

Commit message: Updated Board file, added package variant for battery holder
Parts:
- BAT1: device SparkFun-Electromechanical:BATTCON_20MM_4LEGS_OVERPASTE -> SparkFun-Electromechanical:BATTCON_20MM_4LEGS
Connections:
- net N$2: now also BAT1.NEGATIVE; no longer BAT1.2
- net N$3: now also BAT1.POSITIVE@1, BAT1.POSITIVE@2, BAT1.POSITIVE@3, BAT1.POSITIVE@4; no longer BAT1.1
Routing:
- net N$3: track 41.3 -> 41.2 mm, vias 4 -> 0
