File: Hardware/SparkFun_LilyPad-Switched-Battery_StakingVias_LargePads.sch (EAGLE design)
At the start: 13 parts

Commit message: Updated Board file, added package variant for battery holder
Parts:
- BAT1: device SparkFun-Electromechanical:BATTERY20MM_4LEGS_OVERPASTE -> SparkFun-Electromechanical:BATTERY20MM_4LEGS
Changed lines of the file:
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@@
 <part name="ST4" library="LilyPad-Wearables" deviceset="SEWTAP" device="6"/>
 <part name="U$5" library="LilyPad-Wearables" deviceset="LOGO-LP" device="LP"/>
-<part name="BAT1" library="SparkFun-Electromechanical" deviceset="BATTERY" device="20MM_4LEGS_OVERPASTE" value="20mm coincell"/>
+<part name="BAT1" library="SparkFun-Electromechanical" deviceset="BATTERY" device="20MM_4LEGS" value="20mm coincell"/>
 <part name="U$7" library="SparkFun-Aesthetics" deviceset="OSHW-LOGO" device="S"/>
 <part name="JP1" library="SparkFun-Aesthetics" deviceset="FIDUCIAL" device="UFIDUCIAL"/>
