File: Hardware/Sparkfun_LilyPad-Switched-Battery.sch (EAGLE design)
At the start: 10 parts

Commit message: Updated Brd and Sch files
Other:
- note added: "Jim Lindblom"
- note removed: "L. Buechley, N. Seidle, P. Lewis, T. Klopfenstein"
Changed lines of the file:
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@@
 <plain>
 <circle x="116.84" y="111.76" radius="27.4743" width="0.2032" layer="94"/>
-<text x="165.862" y="11.938" size="1.778" layer="94">L. Buechley, N. Seidle,  P. Lewis, T. Klopfenstein</text>
-<text x="168.402" y="7.112" size="1.778" layer="94">M. West</text>
+<text x="168.402" y="7.112" size="1.778" layer="94" font="vector">M. West</text>
 <text x="238.76" y="7.62" size="1.27" layer="94">v14</text>
+<text x="166.37" y="11.938" size="1.778" layer="94" font="vector">Jim Lindblom</text>
 </plain>
 <instances>

Commit message: Updated Brd and Sch Files
Parts:
- added FD1, FD2: FIDUCIALUFIDUCIAL, SparkFun-Aesthetics:FIDUCIALUFIDUCIAL
Other:
- note added: "v13"
- note removed: "v14"
Changed lines of the file:
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@@
 <part name="LOGO1" library="SparkFun-Aesthetics" deviceset="SFE_LOGO_FLAME" device=".1_INCH" value="SFE_LOGO_FLAME.1_INCH"/>
 <part name="LOGO2" library="SparkFun-Aesthetics" deviceset="OSHW-LOGO" device="S" value="OSHW-LOGOS"/>
+<part name="FD1" library="SparkFun-Aesthetics" deviceset="FIDUCIAL" device="UFIDUCIAL"/>
+<part name="FD2" library="SparkFun-Aesthetics" deviceset="FIDUCIAL" device="UFIDUCIAL"/>
 </parts>
 <sheets>
@@
 <circle x="116.84" y="111.76" radius="27.4743" width="0.2032" layer="94"/>
 <text x="168.402" y="7.112" size="1.778" layer="94" font="vector">M. West</text>
-<text x="238.76" y="7.62" size="1.27" layer="94">v14</text>
+<text x="238.76" y="7.62" size="1.27" layer="94">v13</text>
 <text x="166.37" y="11.938" size="1.778" layer="94" font="vector">Jim Lindblom</text>
 </plain>
@@
 <instance part="LOGO1" gate="G$1" x="213.36" y="40.64"/>
 <instance part="LOGO2" gate="G$1" x="233.68" y="48.26"/>
+<instance part="FD1" gate="G$1" x="226.06" y="27.94"/>
+<instance part="FD2" gate="G$1" x="233.68" y="27.94"/>
 </instances>
 <busses>
